File: circuits/Camera/RS485.kicad_sch (KiCad schematic)
At the start: 19 parts, among them J3 Conn_01x06_MountingPin, J4 Conn_01x06_MountingPin, Q1 S8550, U3 MAX3485, U4 MAX3485

Commit message: すてい
Parts:
- JP3: footprint (none) -> Jumper:SolderJumper-2_P1.3mm_Open_TrianglePad1.0x1.5mm
Changed lines of the file:
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@@
       (effects (font (size 1.27 1.27)))
     )
-    (property "Footprint" "" (at 180.34 139.7 0)
+    (property "Footprint" "Jumper:SolderJumper-2_P1.3mm_Open_TrianglePad1.0x1.5mm" (at 180.34 139.7 0)
       (effects (font (size 1.27 1.27)) hide)
     )
@@
     (pin "1")
     (instances
-      (project "RS485"
-        (path "/37bf7c32-2e7a-419a-b7a7-8c0045b1c536"
-          (reference "JP3") (unit 1)
-        )
-      )
       (project "Camera"
         (path "/68f95e6d-55c3-4b47-aa0e-ac1487e4e50c/e4881d1c-9e9d-45c4-ac15-b5f81dbc6c6f"
