File: circuits/Camera/UI.kicad_sch (KiCad schematic)
At the start: 11 parts, among them SW2 SW_SPST, SW3 SW_SPDT, SW8 SW_SPDT

Commit message: とちゅう
Parts:
- removed C25: 0.1uF, Capacitor_SMD:C_0402_1005Metric, symbol Device:C
- removed D10, D11: Red, LED_SMD:LED_0603_1608Metric_Pad1.05x0.95mm_HandSolder, symbol Device:LED
- removed R59, R60: 1k, Resistor_SMD:R_0402_1005Metric, symbol Device:R
- removed R61, R62, R63: 10k, Resistor_SMD:R_0402_1005Metric, symbol Device:R
- removed SW2: SW_SPST, Button_Switch_SMD:SW_SPST_Omron_B3FS-100xP, symbol Switch:SW_SPST
- removed SW3, SW8: SW_SPDT, MyLibrary:SW_Slide_3P_SPDT, symbol Switch:SW_SPDT
- added C24: 0.1uF, Capacitor_SMD:C_0402_1005Metric, symbol Device:C
- added D8, D9: Red, LED_SMD:LED_0603_1608Metric_Pad1.05x0.95mm_HandSolder, symbol Device:LED
- added R32, R33: 1k, Resistor_SMD:R_0402_1005Metric, symbol Device:R
- added R34, R35, R36: 10k, Resistor_SMD:R_0402_1005Metric, symbol Device:R
- added SW4, SW5: SW_SPDT, MyLibrary:SW_Slide_3P_SPDT, symbol Switch:SW_SPDT
- added SW6: SW_SPST, Button_Switch_SMD:SW_SPST_Omron_B3FS-100xP, symbol Switch:SW_SPST
Connections:
- net +3.3V: now also C24.1, SW4.2 (B), SW5.2 (B), SW6.2 (B)
- net GNDD: now also D8.1 (K), D9.1 (K), R34.2, R35.2, R36.2
- net LED0: now also R32.2
- net LED1: now also R33.2
- net Slide_SW0: now also R35.1, SW4.1 (A)
- net Slide_SW1: now also R36.1, SW5.1 (A)
- net Tact_SW0: now also C24.2, R34.1, SW6.1 (A)
- new net: D9.2 (A), R33.1
- new net: D8.2 (A), R32.1

Commit message: すてい
Parts:
- R32, R33: value 1k -> 2k
Connections:
- net LED0: now also R33.2; no longer R32.2
- net LED1: now also R32.2; no longer R33.2
- net at D9.2 (A): now also R32.1; no longer R33.1
- net at D8.2 (A): now also R33.1; no longer R32.1
Changed lines of the file:
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@@
     (effects (font (size 1.27 1.27)) (justify right))
   )
+  (symbol (lib_id "Device:R") (at 134.62 63.5 270) (mirror x) (unit 1)
+    (in_bom yes) (on_board yes) (dnp no)
+    (property "Reference" "R32" (at 134.62 68.58 90)
+      (effects (font (size 1.27 1.27)))
+    )
+    (property "Value" "2k" (at 134.62 66.04 90)
+      (effects (font (size 1.27 1.27)))
+    )
+    (property "Footprint" "Resistor_SMD:R_0402_1005Metric" (at 134.62 65.278 90)
+      (effects (font (size 1.27 1.27)) hide)
+    )
+    (property "Datasheet" "~" (at 134.62 63.5 0)
+      (effects (font (size 1.27 1.27)) hide)
+    )
+    (pin "1")
+    (pin "2")
+    (instances
+      (project "Camera"
+        (path "/68f95e6d-55c3-4b47-aa0e-ac1487e4e50c/8e34f9fe-cde5-41c5-aa21-c95fd685b9d1"
+          (reference "R32") (unit 1)
+        )
+      )
+    )
+  )
   (symbol (lib_id "Switch:SW_SPST") (at 134.62 91.44 180) (unit 1)
     (in_bom yes) (on_board yes) (dnp no)
@@
         (path "/68f95e6d-55c3-4b47-aa0e-ac1487e4e50c/8e34f9fe-cde5-41c5-aa21-c95fd685b9d1"
           (reference "R34") (unit 1)
-        )
-      )
-    )
-  )
-  (symbol (lib_id "Device:R") (at 134.62 63.5 270) (mirror x) (unit 1)
-    (in_bom yes) (on_board yes) (dnp no)
-    (property "Reference" "R33" (at 134.62 68.58 90)
-      (effects (font (size 1.27 1.27)))
-    )
-    (property "Value" "1k" (at 134.62 66.04 90)
-      (effects (font (size 1.27 1.27)))
-    )
-    (property "Footprint" "Resistor_SMD:R_0402_1005Metric" (at 134.62 65.278 90)
-      (effects (font (size 1.27 1.27)) hide)
-    )
-    (property "Datasheet" "~" (at 134.62 63.5 0)
-      (effects (font (size 1.27 1.27)) hide)
-    )
-    (pin "1")
-    (pin "2")
-    (instances
-      (project "Camera"
-        (path "/68f95e6d-55c3-4b47-aa0e-ac1487e4e50c/8e34f9fe-cde5-41c5-aa21-c95fd685b9d1"
-          (reference "R33") (unit 1)
         )
       )
@@
     )
   )
-  (symbol (lib_id "Device:R") (at 134.62 53.34 270) (mirror x) (unit 1)
-    (in_bom yes) (on_board yes) (dnp no)
-    (property "Reference" "R32" (at 134.62 58.42 90)
-      (effects (font (size 1.27 1.27)))
-    )
-    (property "Value" "1k" (at 134.62 55.88 90)
-      (effects (font (size 1.27 1.27)))
-    )
-    (property "Footprint" "Resistor_SMD:R_0402_1005Metric" (at 134.62 55.118 90)
-      (effects (font (size 1.27 1.27)) hide)
-    )
-    (property "Datasheet" "~" (at 134.62 53.34 0)
-      (effects (font (size 1.27 1.27)) hide)
-    )
-    (pin "1")
-    (pin "2")
-    (instances
-      (project "Camera"
-        (path "/68f95e6d-55c3-4b47-aa0e-ac1487e4e50c/8e34f9fe-cde5-41c5-aa21-c95fd685b9d1"
-          (reference "R32") (unit 1)
-        )
-      )
-    )
-  )
   (symbol (lib_id "power:+3.3V") (at 124.46 91.44 0) (unit 1)
     (in_bom yes) (on_board yes) (dnp no)
@@
         )
       )
+    )
+  )
+  (symbol (lib_id "Device:R") (at 134.62 53.34 270) (mirror x) (unit 1)
+    (in_bom yes) (on_board yes) (dnp no)
+    (property "Reference" "R33" (at 134.62 58.42 90)
+      (effects (font (size 1.27 1.27)))
+    )
+    (property "Value" "2k" (at 134.62 55.88 90)
+      (effects (font (size 1.27 1.27)))
+    )
+    (property "Footprint" "Resistor_SMD:R_0402_1005Metric" (at 134.62 55.118 90)
+      (effects (font (size 1.27 1.27)) hide)
+    )
+    (property "Datasheet" "~" (at 134.62 53.34 0)
+      (effects (font (size 1.27 1.27)) hide)
+    )
+    (pin "1")
+    (pin "2")
+    (instances
+      (project "Camera"
+        (path "/68f95e6d-55c3-4b47-aa0e-ac1487e4e50c/8e34f9fe-cde5-41c5-aa21-c95fd685b9d1"
+          (reference "R33") (unit 1)
+        )
+      )
