File: circuits/Camera/Camera.kicad_sch (KiCad schematic)
At the start: 22 parts, among them J2 Conn_01x14_Pin, SW2 SW_SPST, SW3 SW_SPST, U5 STM32F446RETx, Y1 16MHz, Y2 32.768kHz

Commit message: すてい
Parts:
- removed C15, C16: 22pF, Capacitor_SMD:C_0603_1608Metric, symbol Device:C
- removed SW2: SW_SPST, Button_Switch_SMD:SW_Push_1P1T_NO_Vertical_Wuerth_434133025816, symbol Switch:SW_SPST
- removed Y2: 32.768kHz, Crystal:Crystal_SMD_3215-2Pin_3.2x1.5mm, symbol Device:Crystal
- J2: footprint (none) -> MyLibrary:BoxHeader_2x07_P1.27mm_Horizontal
Connections:
- net GND is gone; now on net GNDD: R37.2
- net MonitorLED0 is gone; now on an unnamed net: R37.1
- net SWCLK: now also U5.49 (PA14)
- net SWDIO: now also U5.46 (PA13)
- net SWO: now also U5.55 (PB3)
- net MainTX4_CamRX: now reaches U5.14 (PA0)
- net MainRX4_CamTX: now reaches U5.15 (PA1)
- net MainTX2_CamRX: now reaches U5.16 (PA2)
- net MainRX2_CamTX: now reaches U5.17 (PA3)
- net MainTX6_CamRX: now reaches U5.37 (PC6)
- net MainRX6_CamTX: now reaches U5.38 (PC7)
- net MainTX1_CamRX: now reaches U5.42 (PA9)
- net MainRX1_CamTX: now reaches U5.43 (PA10)
- net MainTX3_CamRX: now reaches U5.51 (PC10)
- net MainRX3_CamTX: now reaches U5.52 (PC11)
- net MainTX5_CamRX: now reaches U5.53 (PC12)
- net MainRX5_CamTX: now reaches U5.54 (PD2)
- no-connect marks 6 -> 11
Other:
- sheet Cam ports: added MainRX_Cam0TX, MainRX_Cam1TX, MainRX_Cam2TX, MainRX_Cam3TX, MainRX_CamSprTX, MainTX_Cam0RX, MainTX_Cam1RX, MainTX_Cam2RX, MainTX_Cam3RX, MainTX_CamSprRX; removed none
- note added: "マイコン側のラベルと階層シート側のラベルをそれぞれ対応するように書き換える"
- note removed: "LSE"
- moved on the sheet: C11, C12, C13, C14, C17, C18, C19, Y1

Commit message: 修正
Other:
- note added: "マイコン側のラベルと階層シート側のラベルをそれぞれ対応するように書き換える 電解コンの耐圧注意"
- note removed: "マイコン側のラベルと階層シート側のラベルをそれぞれ対応するように書き換える"
Changed lines of the file:
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@@
     (effects (font (size 1.27 1.27)) (justify left bottom))
   )
-  (text "マイコン側のラベルと階層シート側のラベルをそれぞれ対応するように書き換える" (at 17.78 -5.08 0)
+  (text "マイコン側のラベルと階層シート側のラベルをそれぞれ対応するように書き換える\n電解コンの耐圧注意" (at 17.78 -5.08 0)
     (effects (font (size 5.56 5.56)) (justify left bottom))
   )
