File: circuits/Camera/Power.kicad_sch (KiCad schematic)
At the start: 60 parts, among them IC1 DCDC_MPM3620A, IC2 DCDC_MPM3620A, J1 Conn_01x02_Male, Q10 SSM6J808R, Q11 SSM6J808R, Q2 BSS138, Q3 SSM3J332R, Q4 BSS138, Q5 BSS138, Q6 SSM3J332R, SW1 SW_SPDT_White, U1 AZ1117CH-3.3

Commit message: すてい
Parts:
- R19, R20: value 1k -> 2k
Other:
- moved on the sheet: C1, C10, C2, C21, C27, C3, C4, C5, C6, C7, C8, C9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

Commit message: 修正
Other:
- note added: "電源スイッチ 耐圧大丈夫？"
Changed lines of the file:
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@@
     (effects (font (size 1.27 1.27)) (justify left bottom))
+  )
+  (text "電源スイッチ　耐圧大丈夫？" (at 99.06 2.54 0)
+    (effects (font (size 5.56 5.56)) (justify left bottom))
   )
   (text "保護回路・スイッチ" (at 63.5 25.4 0)
