File: circuits/MD/MD.kicad_pcb (KiCad board)
At the start: 2 copper layers, 170 parts, among them IC1 DCDC_MPM3620A, J1 Conn_01x02_Male, J2 Conn_01x10_Male, J7 Conn_01x06_MountingPin, J8 Conn_01x06_MountingPin, Q1 TPH3R704PL, Q10 S8050, Q11 S8050, Q2 TPH3R704PL, Q3 TPH3R704PL, Q4 TPH3R704PL, Q5 TPH3R704PL, Q6 TPH3R704PL, Q7 BSS138, Q8 SSM3J332R, Q9 BSS138, SW1 SW_SPDT_White, SW2 SW_SPST, SW3 SW_SPST, SW5 SW_DIP_x02, U1 Driver_FETGate_DRV8323x, U2 DI035P04PT, U3 DI035P04PT, U4 AZ1117CH-3.3, U5 STM32F446RETx, U6 MAX3485, U7 MAX3485, Y1 16MHz, Y2 32.768kHz

Commit message: とちゅう
Parts:
- removed C22, C34, C35, C36, C37, C38, C39: 0.1uF, Capacitor_SMD:C_0402_1005Metric
- removed J7, J8: Conn_01x06_MountingPin, Connector_Molex:Molex_PicoBlade_53261-0671_1x06-1MP_P1.25mm_Horizontal
- removed Q11: S8050, Package_TO_SOT_SMD:SOT-23
- removed R10, R8, R9: 10k, Resistor_SMD:R_0402_1005Metric
- removed SW5: SW_DIP_x02, Package_DIP:DIP-4_W7.62mm
- removed Y1: 16MHz, Crystal:Crystal_SMD_3225-4Pin_3.2x2.5mm_HandSoldering
- removed Y2: 32.768kHz, Crystal:Crystal_SMD_3215-2Pin_3.2x1.5mm
- added C44: 22pF, Capacitor_SMD:C_0603_1608Metric, F.Cu at (109.0, 36.0)
- added C45: 22pF, Capacitor_SMD:C_0603_1608Metric, F.Cu at (109.0, 38.6)
- added C46: 0.1uF, Capacitor_SMD:C_0402_1005Metric, F.Cu at (98.8, 32.4)
- added C48: 0.1uF, Capacitor_SMD:C_0402_1005Metric, F.Cu at (98.8, 34.4)
- added C50: 0.1uF, Capacitor_SMD:C_0402_1005Metric, F.Cu at (98.8, 36.4)
- added C51: 0.1uF, Capacitor_SMD:C_0402_1005Metric, F.Cu at (98.8, 38.3)
- added C52: 0.1uF, Capacitor_SMD:C_0402_1005Metric, F.Cu at (98.8, 40.3)
- added C53: 0.1uF, Capacitor_SMD:C_0402_1005Metric, F.Cu at (98.8, 42.3)
- added D17: Red, LED_SMD:LED_0603_1608Metric_Pad1.05x0.95mm_HandSolder, F.Cu at (85.2, 35.2)
- added D21: Red, LED_SMD:LED_0603_1608Metric_Pad1.05x0.95mm_HandSolder, F.Cu at (85.2, 37.8)
- added D22: 1N5819WS, Diode_SMD:D_SOD-323_HandSoldering, F.Cu at (109.5, 42.4)
- added J4: Conn_01x06_MountingPin, Connector_Molex:Molex_PicoBlade_53261-0671_1x06-1MP_P1.25mm_Horizontal, F.Cu at (105.1, 18.0)
- added J5: Conn_01x06_MountingPin, Connector_Molex:Molex_PicoBlade_53261-0671_1x06-1MP_P1.25mm_Horizontal, F.Cu at (105.1, 25.8)
- added L1: 22uH, MyLibrary:Inductor_CDPH4D19F, F.Cu at (87.0, 26.5)
- added Q12: DI035P04PT, MyLibrary:Package_TSON-Advance, F.Cu at (86.1, 17.1)
- added Q13: DI035P04PT, MyLibrary:Package_TSON-Advance, F.Cu at (92.3, 17.1)
- added R76: 1k, Resistor_SMD:R_0402_1005Metric, F.Cu at (88.8, 34.9)
- added R77: 10k, Resistor_SMD:R_0402_1005Metric, F.Cu at (88.8, 36.9)
- added R79: 1k, Resistor_SMD:R_0402_1005Metric, F.Cu at (108.4, 44.9)
- added SW4: SW_SPST, Button_Switch_SMD:SW_Push_1P1T_NO_Vertical_Wuerth_434133025816, F.Cu at (103.6, 33.8)
- added SW6: SW_SPST, Button_Switch_SMD:SW_Push_1P1T_NO_Vertical_Wuerth_434133025816, F.Cu at (103.6, 38.6)
- added Y3: 16MHz, Crystal:Crystal_SMD_3225-4Pin_3.2x2.5mm_HandSoldering, F.Cu at (103.6, 43.8)
- added Y4: 32.768kHz, Crystal:Crystal_SMD_3215-2Pin_3.2x1.5mm, F.Cu at (109.5, 33.1)
- C24, C31: value 22pF -> 0.1uF; footprint Capacitor_SMD:C_0603_1608Metric -> Capacitor_SMD:C_0402_1005Metric
- C32, C33: value 22pF -> 1uF; footprint Capacitor_SMD:C_0603_1608Metric -> Capacitor_SMD:C_0402_1005Metric
- C42, C43: value 0.1uF -> 22pF; footprint Capacitor_SMD:C_0402_1005Metric -> Capacitor_SMD:C_0603_1608Metric
- J2: value Conn_01x10_Male -> Conn_01x03_Male; footprint MyLibrary:BoxHeader_2x05_P1.27mm_Vertical_SMD -> Connector_Molex:Molex_SPOX_5268-03A_1x03_P2.50mm_Horizontal
- Q10: value S8050 -> S8550
- R44: footprint Resistor_SMD:R_0402_1005Metric -> Resistor_SMD:R_0603_1608Metric
- R61: value 10k -> 7.5k; footprint Resistor_SMD:R_0402_1005Metric -> Resistor_SMD:R_0603_1608Metric
- R64: value 7.5k -> 10k; footprint Resistor_SMD:R_0603_1608Metric -> Resistor_SMD:R_0402_1005Metric
- R65: value 20k -> 10k
- R66: value 2.2k -> 20k
- R68: value 120 -> 2.2k
- R71: value 7.5k -> 2.2k; footprint Resistor_SMD:R_0603_1608Metric -> Resistor_SMD:R_0402_1005Metric
- R72: value 20k -> 2.2k
- R73, R74: value 2.2k -> 120
- R75: value 120 -> 1k
- SW2: value SW_SPST -> SW_DIP_x02; footprint Button_Switch_SMD:SW_Push_1P1T_NO_Vertical_Wuerth_434133025816 -> Package_DIP:DIP-4_W7.62mm
- SW3: value SW_SPST -> SW_SPDT; footprint Button_Switch_SMD:SW_Push_1P1T_NO_Vertical_Wuerth_434133025816 -> MyLibrary:SW_Slide_3P_SPDT
- U2: value DI035P04PT -> STM32G473CET6; footprint MyLibrary:Package_TSON-Advance -> Package_QFP:LQFP-48_7x7mm_P0.5mm
- U3: value DI035P04PT -> Encoder_Magnetic_AS5047P; footprint MyLibrary:Package_TSON-Advance -> Package_SO:TSSOP-14_4.4x5mm_P0.65mm
- U4: footprint Package_TO_SOT_SMD:TO-252-3_TabPin2 -> Package_TO_SOT_SMD:SOT-223-3_TabPin2
- moved SW3 7.53 mm to (33.0, 55.9)
Connections:
- net /MotorDriver/CAL renamed CAL
- net /MotorDriver/Current_OUTA renamed Current_OUTA
- net /MotorDriver/Current_OUTB renamed Current_OUTB
- net /MotorDriver/Current_OUTC renamed Current_OUTC
- net /MotorDriver/ENABLE renamed ENABLE
- net /MotorDriver/INA_H renamed INA_H
- net /MotorDriver/INA_L renamed INA_L
- net /MotorDriver/INB_H renamed INB_H
- net /MotorDriver/INB_L renamed INB_L
- net /MotorDriver/INC_H renamed INC_H
- net /MotorDriver/INC_L renamed INC_L
- net /MotorDriver/nFAULT renamed nFAULT
- net /Power/V_Measure renamed V_Meas.
- net /Power/Vfb renamed Net-(D20-A)
- net 主電源スイッチ renamed /Power/PowerSW
- C19 pad 2: Net-(U3-G) -> Net-(Q12-G)
- C24 pad 1: GND -> +3.3V
- C24 pad 2: HSE_IN -> GND
- C31 pad 1: GND -> +3.3V
- C31 pad 2: HSE_OUT -> GND
- C32 pad 1: GND -> +3.3V
- C32 pad 2: LSE_IN -> GND
- C33 pad 2: LSE_OUT -> +3.3V
- C42 pad 1: +3.3V -> GND
- C42 pad 2: GND -> HSE_IN
- C43 pad 1: +3.3V -> GND
- C43 pad 2: GND -> HSE_OUT
- J2 pad 1: /3.3VBUS -> /MotorDriver/Phase_U
- J2 pad 2: unconnected-(J2-Pin_2-Pad2) -> /MotorDriver/Phase_V
- J2 pad 3: TCK -> /MotorDriver/Phase_W
- JP1 pad 1: RS485a_A -> /RS485/RS485_A
- JP2 pad 1: RS485a_A -> /RS485/RS485_X
- R42 pad 1: Net-(U2-G) -> Net-(Q13-G)
- R43 pad 2: Net-(U2-G) -> Net-(Q13-G)
- R45 pad 2: Net-(U3-G) -> Net-(Q12-G)
- R46 pad 1: Net-(U3-G) -> Net-(Q12-G)
- R61 pad 1: BOOT0 -> Net-(Q10-B)
- R61 pad 2: GND -> MainTX3_RS485RX
- R64 pad 1: Net-(Q10-B) -> BOOT0
- R64 pad 2: MainTX6_RS485aRX -> GND
- R65 pad 1: Net-(Q10-C) -> Net-(U6-DE)
- R66 pad 1: +3.3V -> Net-(Q10-C)
- R66 pad 2: RS485a_A -> GND
- R67 pad 1: RS485a_B -> +3.3V
- R67 pad 2: GND -> /RS485/RS485_A
- R68 pad 1: Net-(JP1-B) -> /RS485/RS485_B
- R68 pad 2: RS485a_B -> GND
- R69 pad 2: DIP_SW0 -> /UI/DIP_SW0
- R70 pad 2: DIP_SW1 -> /UI/DIP_SW1
- R71 pad 1: Net-(Q11-B) -> +3.3V
- R71 pad 2: MainTX6_RS485aRX -> /RS485/RS485_X
- R72 pad 1: Net-(Q11-C) -> /RS485/RS485_Y
- R73 pad 1: +3.3V -> Net-(JP1-B)
- R73 pad 2: RS485a_A -> /RS485/RS485_B
- R74 pad 1: RS485a_B -> Net-(JP2-B)
- R74 pad 2: GND -> /RS485/RS485_Y
- R75 pad 1: Net-(JP2-B) -> Net-(D17-A)
- R75 pad 2: RS485a_B -> /UI/LED0
- SW2 pad 1: BOOT0 -> /UI/DIP_SW0
- SW2 pad 2: +3.3V -> /UI/DIP_SW1
- SW3 pad 1: NRST -> /UI/Slide_SW0
- SW3 pad 2: GND -> +3.3V
- U2 pad 1: /Power/24VBAT -> +3.3V
- U2 pad 2: /Power/24VBAT -> unconnected-(U2-PC13-Pad2)
- U2 pad 3: /Power/24VBAT -> unconnected-(U2-PC14-Pad3)
- U2 pad 4: Net-(U2-G) -> unconnected-(U2-PC15-Pad4)
- U2 pad 5: /Power/S-S -> unconnected-(U2-PF0-Pad5)
- U3 pad 1: VDD -> /Encoder/CS
- U3 pad 2: VDD -> /Encoder/CLK
- U3 pad 3: VDD -> /Encoder/MISO
- U3 pad 4: Net-(U3-G) -> /Encoder/MOSI
- U3 pad 5: /Power/S-S -> GND
- U6 pad 1: MainRX6_RS485aTX -> MainRX3_RS485TX
- U6 pad 2: Net-(Q10-C) -> Net-(U6-DE)
- U6 pad 3: Net-(Q10-C) -> Net-(U6-DE)
- U6 pad 4: MainTX6_RS485aRX -> unconnected-(U6-DI-Pad4)
- U6 pad 6: RS485a_A -> /RS485/RS485_A
- U6 pad 7: RS485a_B -> /RS485/RS485_B
- U7 pad 1: MainRX6_RS485aTX -> unconnected-(U7-RO-Pad1)
- U7 pad 2: Net-(Q11-C) -> Net-(Q10-C)
- U7 pad 3: Net-(Q11-C) -> Net-(Q10-C)
- U7 pad 4: MainTX6_RS485aRX -> MainTX3_RS485RX
- U7 pad 6: RS485a_A -> /RS485/RS485_X
- U7 pad 7: RS485a_B -> /RS485/RS485_Y

Commit message: すてい
Parts:
- removed C40: 4.7uF, Capacitor_SMD:C_0603_1608Metric
- removed C41: 1uF, Capacitor_SMD:C_0402_1005Metric
- removed C44, C45: 22pF, Capacitor_SMD:C_0603_1608Metric
- removed Q3, Q4, Q5, Q6: TPH3R704PL, MyLibrary:Package_TSON-Advance
- removed R63: 10k, Resistor_SMD:R_0402_1005Metric
- removed R75, R76: 1k, Resistor_SMD:R_0402_1005Metric
- removed SW4: SW_SPST, Button_Switch_SMD:SW_Push_1P1T_NO_Vertical_Wuerth_434133025816
- removed U5: STM32F446RETx, Package_QFP:LQFP-64_10x10mm_P0.5mm
- removed Y4: 32.768kHz, Crystal:Crystal_SMD_3215-2Pin_3.2x1.5mm
- added C22: 4.7uF, Capacitor_SMD:C_0603_1608Metric, F.Cu at (96.6, 49.1)
- added J3: Conn_01x14_Pin, MyLibrary:BoxHeader_2x07_P1.27mm_Horizontal, F.Cu at (78.2, 91.0)
- added JP3: SolderJumper_2_Open, Jumper:SolderJumper-2_P1.3mm_Open_TrianglePad1.0x1.5mm, F.Cu at (90.7, 83.8)
- added Q14: DMT6017LDV, MyLibrary:Package_TSON-Advance_DualFET, F.Cu at (93.0, 69.1)
- added R10: 2k, Resistor_SMD:R_0402_1005Metric, F.Cu at (96.0, 53.3)
- added R8: 2k, Resistor_SMD:R_0402_1005Metric, F.Cu at (91.1, 48.8)
- added R9: 2k, Resistor_SMD:R_0402_1005Metric, F.Cu at (91.1, 50.8)
- C1: value 22uF -> 10uF; footprint Capacitor_SMD:C_0402_1005Metric -> Capacitor_SMD:C_1206_3216Metric
- C32: value 1uF -> 10uF; footprint Capacitor_SMD:C_0402_1005Metric -> Capacitor_SMD:C_1206_3216Metric
- C5: footprint Capacitor_SMD:C_0402_1005Metric -> Capacitor_SMD:C_0603_1608Metric
- C7, C8, C9: value 30pF -> 330pF; footprint Capacitor_SMD:C_0402_1005Metric -> Capacitor_SMD:C_0603_1608Metric
- Q1, Q2: value TPH3R704PL -> DMT6017LDV; footprint MyLibrary:Package_TSON-Advance -> MyLibrary:Package_TSON-Advance_DualFET
- R1: value 10k -> 1k
- R15, R16, R17: value 1k -> 100
- R22, R27, R32: value 20mR -> 7m
- R35, R38, R41: value 10k -> 20k
- R54: value 1k -> 2k
- R55: value 1k -> 10k
- U1: value Driver_FETGate_DRV8323x -> Driver_FETGate_DRV8323S
Connections:
- net /MotorDriver/nSCS renamed CS1_MD
- C32 pad 1: +3.3V -> VDD
- Q1 pad 1: /MotorDriver/Phase_U -> Net-(D8-A)
- Q1 pad 2: /MotorDriver/Phase_U -> Net-(Q1A-G)
- Q1 pad 3: /MotorDriver/Phase_U -> /MotorDriver/Phase_V
- Q1 pad 4: Net-(Q1-G) -> Net-(Q1B-G)
- Q2 pad 1: Net-(D6-A) -> Net-(D10-A)
- Q2 pad 2: Net-(D6-A) -> Net-(Q2A-G)
- Q2 pad 3: Net-(D6-A) -> /MotorDriver/Phase_W
- Q2 pad 4: Net-(Q2-G) -> Net-(Q2B-G)
- Q2 pad 5: /MotorDriver/Phase_U -> VDD
- R13 pad 1: /MotorDriver/SDO -> MISO1
- R18 pad 2: Net-(Q1-G) -> Net-(Q14B-G)
- R19 pad 2: Net-(Q2-G) -> Net-(Q14A-G)
- R20 pad 1: Net-(Q1-G) -> Net-(Q14B-G)
- R21 pad 1: Net-(Q2-G) -> Net-(Q14A-G)
- R23 pad 2: Net-(Q3-G) -> Net-(Q1B-G)
- R24 pad 2: Net-(Q4-G) -> Net-(Q1A-G)
- R25 pad 2: Net-(Q3-G) -> Net-(Q1B-G)
- R26 pad 2: Net-(Q4-G) -> Net-(Q1A-G)
- R28 pad 2: Net-(Q5-G) -> Net-(Q2B-G)
- R29 pad 2: Net-(Q6-G) -> Net-(Q2A-G)
- R30 pad 2: Net-(Q5-G) -> Net-(Q2B-G)
- R31 pad 2: Net-(Q6-G) -> Net-(Q2A-G)
- R35 pad 1: Net-(D11-A) -> /MotorDriver/Phase_U
- R35 pad 2: /MotorDriver/Phase_U -> Net-(D11-A)
- R38 pad 1: Net-(D12-A) -> /MotorDriver/Phase_V
- R38 pad 2: /MotorDriver/Phase_V -> Net-(D12-A)
- R41 pad 1: Net-(D13-A) -> /MotorDriver/Phase_W
- R41 pad 2: /MotorDriver/Phase_W -> Net-(D13-A)
- R54 pad 1: Net-(D18-A) -> Net-(D17-A)
- R54 pad 2: +5V -> /UI/LED0
- R55 pad 1: Net-(D19-A) -> Net-(U2-PB2)
- R55 pad 2: +3.3V -> GND
- U1 pad 26: /MotorDriver/SDO -> MISO1
- U1 pad 27: /MotorDriver/SDI -> MOSI1
- U1 pad 28: /MotorDriver/SCLK -> SCLK1
- U2 pad 10: unconnected-(U2-PA2-Pad10) -> Current_OUTC
- U2 pad 11: unconnected-(U2-PA3-Pad11) -> V_Meas.
- U2 pad 13: unconnected-(U2-PA5-Pad13) -> SCLK1
- U2 pad 14: unconnected-(U2-PA6-Pad14) -> MISO1
- U2 pad 15: unconnected-(U2-PA7-Pad15) -> MOSI1
- U2 pad 18: unconnected-(U2-PB2-Pad18) -> Net-(U2-PB2)
- U2 pad 22: unconnected-(U2-PB10-Pad22) -> MainTX3_RS485RX
- U2 pad 25: unconnected-(U2-PB11-Pad25) -> MainRX3_RS485TX
- U2 pad 37: unconnected-(U2-PA13-Pad37) -> SWDIO
- U2 pad 38: unconnected-(U2-PA14-Pad38) -> SWCLK
- U2 pad 40: unconnected-(U2-PB3-Pad40) -> SWO
- U2 pad 45: unconnected-(U2-PB8-BOOT0-Pad45) -> BOOT0
- U2 pad 5: unconnected-(U2-PF0-Pad5) -> HSE_IN
- U2 pad 6: unconnected-(U2-PF1-Pad6) -> HSE_OUT
- U2 pad 7: unconnected-(U2-NRST-Pad7) -> NRST
- U2 pad 8: unconnected-(U2-PA0-Pad8) -> Current_OUTA
- U2 pad 9: unconnected-(U2-PA1-Pad9) -> Current_OUTB
