File: circuits/MD/Power.kicad_sch (KiCad schematic)
At the start: 48 parts, among them IC1 DCDC_MPM3620A, J1 Conn_01x02_Male, Q12 DI035P04PT, Q13 DI035P04PT, Q7 BSS138, Q8 SSM3J332R, Q9 BSS138, SW1 SW_SPDT_White, U4 AZ1117CH-3.3

Commit message: こみっと
Connections:
- net V_Measure renamed V_Meas.
- net Vfb: no longer names the net of C29.1, D20.2 (A), IC1.9 (OUT), Q8.2 (S), R58.2, R60.1
- net 主電源スイッチ renamed PowerSW
Other:
- note added: "スイッチのフットプリント"
Changed lines of the file:
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@@
+    (stroke (width 0) (type default))
+  )
+  (wire (pts (xy 114.3 71.12) (xy 116.84 71.12))
     (stroke (width 0) (type default))
   )
@@
     (stroke (width 0.5) (type solid))
   )
-  (wire (pts (xy 43.18 78.74) (xy 40.64 78.74))
+  (wire (pts (xy 45.72 78.74) (xy 40.64 78.74))
     (stroke (width 0) (type default))
   )
@@
     (stroke (width 0) (type default))
   )
-  (wire (pts (xy 91.44 119.38) (xy 91.44 121.92))
-    (stroke (width 0) (type default))
-  )
   (wire (pts (xy 220.98 78.74) (xy 220.98 80.01))
     (stroke (width 0) (type default))
@@
     (effects (font (size 1.27 1.27)) (justify left bottom))
   )
+  (text "スイッチのフットプリント" (at 121.92 7.62 0)
+    (effects (font (size 5.56 5.56)) (justify left bottom))
+  )
   (text "インジケーターLED" (at 231.14 111.76 0)
     (effects (font (size 1.27 1.27)) (justify left bottom))
@@
   )
   (label "S-S" (at 104.14 43.18 0) (fields_autoplaced)
-    (effects (font (size 1.27 1.27)) (justify left bottom))
+    (effects (font (size 1.27 1.27) (thickness 0.254) bold) (justify left bottom))
   )
   (label "24VBAT" (at 48.26 38.1 0) (fields_autoplaced)
-    (effects (font (size 1.27 1.27)) (justify left bottom))
-  )
-  (label "Vfb" (at 91.44 119.38 0) (fields_autoplaced)
-    (effects (font (size 1.27 1.27)) (justify left bottom))
+    (effects (font (size 1.27 1.27) (thickness 0.254) bold) (justify left bottom))
   )
   (label "S-S" (at 38.1 55.88 0) (fields_autoplaced)
-    (effects (font (size 1.27 1.27)) (justify left bottom))
+    (effects (font (size 1.27 1.27) (thickness 0.254) bold) (justify left bottom))
   )
   (label "PG" (at 96.52 142.24 180) (fields_autoplaced)
@@
   )
   (label "24VBAT" (at 83.82 43.18 180) (fields_autoplaced)
-    (effects (font (size 1.27 1.27)) (justify right bottom))
+    (effects (font (size 1.27 1.27) (thickness 0.254) bold) (justify right bottom))
+  )
+  (label "PowerSW" (at 114.3 71.12 180) (fields_autoplaced)
+    (effects (font (size 1.27 1.27) (thickness 0.254) bold) (justify right bottom))
   )
   (label "PG" (at 78.74 142.24 0) (fields_autoplaced)
     (effects (font (size 1.27 1.27)) (justify left bottom))
   )
-  (global_label "主電源スイッチ" (shape output) (at 43.18 78.74 0) (fields_autoplaced)
-    (effects (font (size 1.27 1.27)) (justify left))
-    (property "Intersheetrefs" "${INTERSHEET_REFS}" (at 57.1116 78.74 0)
-      (effects (font (size 1.27 1.27)) (justify left) hide)
-    )
-  )
-  (global_label "主電源スイッチ" (shape output) (at 116.84 71.12 180) (fields_autoplaced)
-    (effects (font (size 1.27 1.27)) (justify right))
-    (property "Intersheetrefs" "${INTERSHEET_REFS}" (at 103.4807 71.0406 0)
-      (effects (font (size 1.27 1.27)) (justify right) hide)
-    )
-  )
-  (hierarchical_label "V_Measure" (shape input) (at 241.3 38.1 0) (fields_autoplaced)
+  (label "PowerSW" (at 45.72 78.74 0) (fields_autoplaced)
+    (effects (font (size 1.27 1.27) (thickness 0.254) bold) (justify left bottom))
+  )
+  (hierarchical_label "V_Meas." (shape input) (at 241.3 38.1 0) (fields_autoplaced)
     (effects (font (size 1.27 1.27)) (justify left))
   )
@@
   (symbol (lib_name "Q_NMOS_GSD_1") (lib_id "Device:Q_NMOS_GSD") (at 121.92 71.12 0) (unit 1)
     (in_bom yes) (on_board yes) (dnp no)
-    (property "Reference" "Q7" (at 114.3 66.04 0)
-      (effects (font (size 1.27 1.27)) (justify left))
-    )
-    (property "Value" "BSS138" (at 114.3 68.58 0)
-      (effects (font (size 1.27 1.27)) (justify left))
-    )
+    (property "Reference" "Q7" (at 114.3 73.66 0)
+      (effects (font (size 1.27 1.27)) (justify left))
+    )
+    (property "Value" "BSS138" (at 114.3 76.2 0)
+      (effects (font (size 1.27 1.27)) (justify left))
+    )

Commit message: すてい
Parts:
- removed R54, R55: 1k, Resistor_SMD:R_0402_1005Metric, symbol Device:R
- added R8, R9: 2k, Resistor_SMD:R_0402_1005Metric, symbol Device:R
Connections:
- net +3.3V: now also R8.2
- net +5V: now also R9.2
- net at D19.2 (A): now also R8.1
- net at D18.2 (A): now also R9.1
Changed lines of the file:
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@@
     (effects (font (size 1.27 1.27)) (justify left bottom))
   )
-  (text "スイッチのフットプリント" (at 121.92 7.62 0)
+  (text "スイッチのフットプリント" (at 121.92 17.78 0)
     (effects (font (size 5.56 5.56)) (justify left bottom))
   )
@@
     )
   )
-  (symbol (lib_id "Device:R") (at 246.38 142.24 270) (mirror x) (unit 1)
-    (in_bom yes) (on_board yes) (dnp no)
-    (property "Reference" "R55" (at 246.38 147.32 90)
-      (effects (font (size 1.27 1.27)))
-    )
-    (property "Value" "1k" (at 246.38 144.78 90)
-      (effects (font (size 1.27 1.27)))
-    )
-    (property "Footprint" "Resistor_SMD:R_0402_1005Metric" (at 246.38 144.018 90)
-      (effects (font (size 1.27 1.27)) hide)
-    )
-    (property "Datasheet" "~" (at 246.38 142.24 0)
-      (effects (font (size 1.27 1.27)) hide)
-    )
-    (pin "1")
-    (pin "2")
-    (instances
-      (project "MD"
-        (path "/6b908e7d-66d4-4b9c-9a00-1a873c360635/9d25c103-4e41-4e92-b98a-56b88403a364"
-          (reference "R55") (unit 1)
-        )
-      )
-    )
-  )
   (symbol (lib_id "power:VCC") (at 27.94 119.38 0) (unit 1)
     (in_bom yes) (on_board yes) (dnp no)
@@
     )
   )
-  (symbol (lib_id "Device:R") (at 246.38 129.54 270) (mirror x) (unit 1)
-    (in_bom yes) (on_board yes) (dnp no)
-    (property "Reference" "R54" (at 246.38 134.62 90)
-      (effects (font (size 1.27 1.27)))
-    )
-    (property "Value" "1k" (at 246.38 132.08 90)
-      (effects (font (size 1.27 1.27)))
-    )
-    (property "Footprint" "Resistor_SMD:R_0402_1005Metric" (at 246.38 131.318 90)
-      (effects (font (size 1.27 1.27)) hide)
-    )
-    (property "Datasheet" "~" (at 246.38 129.54 0)
-      (effects (font (size 1.27 1.27)) hide)
-    )
-    (pin "1")
-    (pin "2")
-    (instances
-      (project "MD"
-        (path "/6b908e7d-66d4-4b9c-9a00-1a873c360635/9d25c103-4e41-4e92-b98a-56b88403a364"
-          (reference "R54") (unit 1)
-        )
-      )
-    )
-  )
   (symbol (lib_id "Device:R") (at 83.82 142.24 180) (unit 1)
     (in_bom yes) (on_board yes) (dnp no)
@@
     )
   )
+  (symbol (lib_id "Device:R") (at 246.38 142.24 270) (mirror x) (unit 1)
+    (in_bom yes) (on_board yes) (dnp no)
+    (property "Reference" "R8" (at 246.38 147.32 90)
+      (effects (font (size 1.27 1.27)))
+    )
+    (property "Value" "2k" (at 246.38 144.78 90)
+      (effects (font (size 1.27 1.27)))
+    )
+    (property "Footprint" "Resistor_SMD:R_0402_1005Metric" (at 246.38 144.018 90)
+      (effects (font (size 1.27 1.27)) hide)
+    )
+    (property "Datasheet" "~" (at 246.38 142.24 0)
+      (effects (font (size 1.27 1.27)) hide)
+    )
+    (pin "1")
+    (pin "2")
+    (instances
+      (project "MD"
+        (path "/6b908e7d-66d4-4b9c-9a00-1a873c360635/9d25c103-4e41-4e92-b98a-56b88403a364"
+          (reference "R8") (unit 1)
+        )
+      )
+    )
+  )
   (symbol (lib_id "Device:C_Polarized") (at 208.28 83.82 0) (unit 1)
     (in_bom yes) (on_board yes) (dnp no)
@@
         )
       )
+    )
+  )
+  (symbol (lib_id "Device:R") (at 246.38 129.54 270) (mirror x) (unit 1)
+    (in_bom yes) (on_board yes) (dnp no)
+    (property "Reference" "R9" (at 246.38 134.62 90)
+      (effects (font (size 1.27 1.27)))
+    )
+    (property "Value" "2k" (at 246.38 132.08 90)
+      (effects (font (size 1.27 1.27)))
+    )
+    (property "Footprint" "Resistor_SMD:R_0402_1005Metric" (at 246.38 131.318 90)
+      (effects (font (size 1.27 1.27)) hide)
+    )
+    (property "Datasheet" "~" (at 246.38 129.54 0)
+      (effects (font (size 1.27 1.27)) hide)
+    )
+    (pin "1")
+    (pin "2")
+    (instances
+      (project "MD"
+        (path "/6b908e7d-66d4-4b9c-9a00-1a873c360635/9d25c103-4e41-4e92-b98a-56b88403a364"
+          (reference "R9") (unit 1)
+        )
+      )
