File: circuits/MD/RS485.kicad_sch (KiCad schematic)
At the start: 19 parts, among them J4 Conn_01x06_MountingPin, J5 Conn_01x06_MountingPin, Q10 S8550, U6 MAX3485, U7 MAX3485

Commit message: とちゅう
Other:
- note added: "RS485/Device"
- note removed: "RS485"
Changed lines of the file:
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@@
     (fill (type none))
   )
-  (text "RS485" (at 73.66 30.48 0)
+  (text "RS485/Device" (at 73.66 30.48 0)
     (effects (font (size 2.54 2.54) (thickness 0.254) bold) (justify left bottom))
   )

Commit message: すてい
Parts:
- JP3: footprint (none) -> Jumper:SolderJumper-2_P1.3mm_Open_TrianglePad1.0x1.5mm
Changed lines of the file:
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@@
       (effects (font (size 1.27 1.27)))
     )
-    (property "Footprint" "" (at 182.88 142.24 0)
+    (property "Footprint" "Jumper:SolderJumper-2_P1.3mm_Open_TrianglePad1.0x1.5mm" (at 182.88 142.24 0)
       (effects (font (size 1.27 1.27)) hide)
     )
