File: circuits/MD/UI.kicad_sch (KiCad schematic)
At the start: 9 parts, among them SW2 SW_DIP_x02, SW3 SW_SPDT

Commit message: とちゅう
Parts:
- SW3: footprint Slide_Switch:3P_SPDT_SlideSwitch -> MyLibrary:SW_Slide_3P_SPDT
Changed lines of the file:
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@@
       (effects (font (size 1.27 1.27)) (justify left))
     )
-    (property "Footprint" "Slide_Switch:3P_SPDT_SlideSwitch" (at 142.24 134.62 0)
+    (property "Footprint" "MyLibrary:SW_Slide_3P_SPDT" (at 142.24 134.62 0)
       (effects (font (size 1.27 1.27)) hide)
     )

Commit message: すてい
Parts:
- removed R75, R76: 1k, Resistor_SMD:R_0402_1005Metric, symbol Device:R
- added R10, R54: 2k, Resistor_SMD:R_0402_1005Metric, symbol Device:R
Connections:
- net LED0: now also R54.2
- net LED1: now also R10.2
- net at D17.2 (A): now also R54.1
- net at D21.2 (A): now also R10.1
Changed lines of the file:
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@@
   (symbol (lib_id "Device:R") (at 144.78 71.12 270) (mirror x) (unit 1)
     (in_bom yes) (on_board yes) (dnp no)
-    (property "Reference" "R76" (at 144.78 76.2 90)
+    (property "Reference" "R10" (at 144.78 76.2 90)
       (effects (font (size 1.27 1.27)))
     )
-    (property "Value" "1k" (at 144.78 73.66 90)
+    (property "Value" "2k" (at 144.78 73.66 90)
       (effects (font (size 1.27 1.27)))
     )
@@
       (project "MD"
         (path "/6b908e7d-66d4-4b9c-9a00-1a873c360635/95721a70-6e46-4ff1-892b-e4afe28b54e0"
-          (reference "R76") (unit 1)
+          (reference "R10") (unit 1)
         )
       )
@@
   (symbol (lib_id "Device:R") (at 144.78 60.96 270) (mirror x) (unit 1)
     (in_bom yes) (on_board yes) (dnp no)
-    (property "Reference" "R75" (at 144.78 66.04 90)
+    (property "Reference" "R54" (at 144.78 66.04 90)
       (effects (font (size 1.27 1.27)))
     )
-    (property "Value" "1k" (at 144.78 63.5 90)
+    (property "Value" "2k" (at 144.78 63.5 90)
       (effects (font (size 1.27 1.27)))
     )
@@
       (project "MD"
         (path "/6b908e7d-66d4-4b9c-9a00-1a873c360635/95721a70-6e46-4ff1-892b-e4afe28b54e0"
-          (reference "R75") (unit 1)
+          (reference "R54") (unit 1)
         )
       )
