File: circuits/MD/MotorDriver.kicad_sch (KiCad schematic)
At the start: 79 parts, among them Q1 TPH3R704PL, Q2 TPH3R704PL, Q3 TPH3R704PL, Q4 TPH3R704PL, Q5 TPH3R704PL, Q6 TPH3R704PL, U1 Driver_FETGate_DRV8323x

Commit message: こみっと
Parts:
- removed R10, R8, R9: 10k, Resistor_SMD:R_0402_1005Metric, symbol Device:R
- added J2: Conn_01x03_Male, Connector_Molex:Molex_SPOX_5268-03A_1x03_P2.50mm_Horizontal, symbol Connector:Conn_01x03_Male
Connections:
- net Phase_U: now also J2.1 (Pin_1)
- net Phase_V: now also J2.2 (Pin_2)
- net Phase_W: now also J2.3 (Pin_3)
Other:
- note added: "PowerModule"
- note added: "電流センスアンプは差動電圧はどこまでいけるのか？電流最大値の設計 ハーフブリッジFETかえる"
- note removed: "電流センスアンプは差動電圧はどこまでいけるのか？電流最大値の設計"
- moved on the sheet: C1, C10, C11, C12, C13, C14, C15, C16, C17, C18, C2, C3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

Commit message: すてい
Parts:
- removed Q1, Q2, Q3, Q4, Q5, Q6: TPH3R704PL, MyLibrary:Package_TSON-Advance, symbol Transistor_FET:FDMS8050
- added C32: 10uF, Capacitor_SMD:C_1206_3216Metric, symbol Device:C
- added Q1, Q14, Q2: DMT6017LDV, MyLibrary:Package_TSON-Advance_DualFET, symbol Device:Q_Dual_NMOS_S1G1S2G2D2D2D1D1
- C1: value 22uF -> 10uF; footprint Capacitor_SMD:C_0402_1005Metric -> Capacitor_SMD:C_1206_3216Metric
- C5: footprint Capacitor_SMD:C_0402_1005Metric -> Capacitor_SMD:C_0603_1608Metric
- C7, C8, C9: value 30pF -> 330pF; footprint Capacitor_SMD:C_0402_1005Metric -> Capacitor_SMD:C_0603_1608Metric
- R1: value 10k -> 1k
- R15, R16, R17: value 1k -> 100
- R22, R27, R32: value 20mR -> 7m
- R35, R38, R41: value 10k -> 20k
- U1: value Driver_FETGate_DRV8323x -> Driver_FETGate_DRV8323S
Connections:
- net GNDD: now also C32.2
- net Phase_U: now also R35.1, Q14.3 (S), Q14.7 (D), Q14.8 (D); no longer R35.2
- net Phase_V: now also R38.1, Q1.3 (S), Q1.7 (D), Q1.8 (D); no longer R38.2
- net Phase_W: now also R41.1, Q2.3 (S), Q2.7 (D), Q2.8 (D); no longer R41.2
- net VDD: now also C32.1, Q1.5 (D), Q1.6 (D), Q14.5 (D), Q14.6 (D), Q2.5 (D), Q2.6 (D)
- net at D10.2 (A), R31.1, R32.2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: now also Q2.1 (S)
- net at R19.2, R21.1: now also Q14.2 (G)
- net at R18.2, R20.1: now also Q14.4 (G)
- net at R28.2, R30.2: now also Q2.4 (G)
- net at D8.2 (A), R26.1, R27.2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: now also Q1.1 (S)
- net at R29.2, R31.2: now also Q2.2 (G)
- net at D11.2 (A): now also R35.2; no longer R35.1
- net at R23.2, R25.2: now also Q1.4 (G)
- net at R24.2, R26.2: now also Q1.2 (G)
- net at D13.2 (A): now also R41.2; no longer R41.1
- net at D12.2 (A): now also R38.2; no longer R38.1
- net at D6.2 (A), R21.2, R22.2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: now also Q14.1 (S)
Other:
- note added: "MotorDriver"
- note added: "試作基板はフィルタのフットプリント0603にする"
- note removed: "PowerModule"
- note removed: "電流センスアンプは差動電圧はどこまでいけるのか？電流最大値の設計 ハーフブリッジFETかえる"
