File: circuits/Main/Mouse.kicad_sch (KiCad schematic)
At the start: 0 parts

Commit message: とちゅう
Parts:
- added C26: 1uF, Capacitor_SMD:C_0402_1005Metric, symbol Device:C
- added Q11: BSS138, Package_TO_SOT_SMD:SOT-23, symbol Device:Q_NMOS_GSD
- added R64: 10k, Resistor_SMD:R_0402_1005Metric, symbol Device:R
- added U10: Sensor_OpticalFlowSensor_PIM453, MyLibrary:Sensor_OpticalFlowSensor_PIM453, symbol MyLibrary:Sensor_OpticalFlowSensor_PIM453
Connections:
- new net: Q11.3 (D), U10.6 (INT)
- new net +3.3V: C26.2, U10.1 (3-5V)
- new net CLK: U10.3 (SCK)
- new net CS: U10.2 (CS)
- new net GNDD: C26.1, Q11.2 (S), R64.2, U10.7 (GND)
- new net MISO: U10.5 (MISO)
- new net MOSI: U10.4 (MOSI)
- new net Mouse_INT: Q11.1 (G), R64.1
Other:
- note added: "マウスセンサー"

Commit message: すてい
Parts:
- removed Q11: BSS138, Package_TO_SOT_SMD:SOT-23, symbol Device:Q_NMOS_GSD
- removed R64: 10k, Resistor_SMD:R_0402_1005Metric, symbol Device:R
- added JP16: SolderJumper_2_Open, Jumper:SolderJumper-2_P1.3mm_Open_TrianglePad1.0x1.5mm, symbol Jumper:SolderJumper_2_Open
Connections:
- net Mouse_INT: now also JP16.1 (A)
- net at U10.6 (INT): now also JP16.2 (B)
Other:
- moved on the sheet: C26, U10
