File: circuits/Main/RS485.kicad_sch (KiCad schematic)
At the start: 95 parts, among them J2 Conn_01x06_MountingPin, J3 Conn_01x06_MountingPin, J4 Conn_01x06_MountingPin, J5 Conn_01x06_MountingPin, J6 Conn_01x06_MountingPin, Q10 S8050, Q11 S8050, Q12 S8050, Q13 S8050, Q14 S8050, Q15 S8050, Q6 S8050, Q7 S8050, Q8 S8050, Q9 S8050, U10 MAX3485, U11 MAX3485, U2 MAX3485, U3 MAX3485, U4 MAX3485, U5 MAX3485, U6 MAX3485, U7 MAX3485, U8 MAX3485, U9 MAX3485

Commit message: こみっと
Parts:
- removed C19, C20: 0.1uF, Capacitor_SMD:C_0402_1005Metric, symbol Device:C
- removed J6: Conn_01x06_MountingPin, Connector_Molex:Molex_PicoBlade_53398-0671_1x06-1MP_P1.25mm_Vertical, symbol Connector_Generic_MountingPin:Conn_01x06_MountingPin
- removed JP1, JP10, JP4, JP7: Jumper_2_Open, Connector_PinHeader_2.54mm:PinHeader_1x02_P2.54mm_Vertical, symbol Jumper:Jumper_2_Open
- removed Q10, Q11, Q12, Q13, Q14, Q15: S8050, Package_TO_SOT_SMD:SOT-23, symbol Device:Q_PNP_BEC
- removed R57, R58, R65, R66, R67, R68: 2.2k, Resistor_SMD:R_0402_1005Metric, symbol Device:R
- removed R59, R60, R69, R70: 120, Resistor_SMD:R_0402_1005Metric, symbol Device:R
- removed R61, R62: 7.5k, Resistor_SMD:R_0603_1608Metric, symbol Device:R
- removed R63, R64: 20k, Resistor_SMD:R_0402_1005Metric, symbol Device:R
- removed U10, U11: MAX3485, Package_SO:SOP-8_3.9x4.9mm_P1.27mm, symbol Interface_UART:MAX3485
- added C21, C22: 0.1uF, Capacitor_SMD:C_0402_1005Metric, symbol Device:C
- added J8: Conn_01x06_MountingPin, Connector_Molex:Molex_PicoBlade_53261-0671_1x06-1MP_P1.25mm_Horizontal, symbol Connector_Generic_MountingPin:Conn_01x06_MountingPin
- added JP1, JP10, JP15, JP4, JP7: SolderJumper_2_Open, symbol Jumper:SolderJumper_2_Open
- added JP11, JP12, JP13, JP14: Jumper_2_Open, Connector_PinHeader_2.54mm:PinHeader_1x02_P2.54mm_Vertical, symbol Jumper:Jumper_2_Open
- added Q5: S8550, Package_TO_SOT_SMD:SOT-23, symbol Device:Q_PNP_BEC
- added R71: 7.5k, Resistor_SMD:R_0603_1608Metric, symbol Device:R
- added R77: 10k, Resistor_SMD:R_0402_1005Metric, symbol Device:R
- added R78: 20k, Resistor_SMD:R_0402_1005Metric, symbol Device:R
- added R79, R80, R87, R88: 2.2k, Resistor_SMD:R_0402_1005Metric, symbol Device:R
- added R89, R90: 120, Resistor_SMD:R_0402_1005Metric, symbol Device:R
- added U14, U16: MAX3485, Package_SO:SOP-8_3.9x4.9mm_P1.27mm, symbol Interface_UART:MAX3485
- J2, J3, J4, J5: footprint Connector_Molex:Molex_PicoBlade_53398-0671_1x06-1MP_P1.25mm_Vertical -> Connector_Molex:Molex_PicoBlade_53261-0671_1x06-1MP_P1.25mm_Horizontal
- Q6, Q7, Q8, Q9: value S8050 -> S8550
- R23: value 2.2k -> 10k
- R25: value 120 -> 2.2k
- R26, R42, R51, R52: value 7.5k -> 2.2k; footprint Resistor_SMD:R_0603_1608Metric -> Resistor_SMD:R_0402_1005Metric
- R27, R33, R34, R43, R44, R53, R54: value 20k -> 2.2k
- R28, R29, R37, R38, R46, R47, R55, R56: value 2.2k -> 120
- R30, R39: value 120 -> 7.5k; footprint Resistor_SMD:R_0402_1005Metric -> Resistor_SMD:R_0603_1608Metric
- R31: value 7.5k -> 20k; footprint Resistor_SMD:R_0603_1608Metric -> Resistor_SMD:R_0402_1005Metric
- R32, R41: value 7.5k -> 10k; footprint Resistor_SMD:R_0603_1608Metric -> Resistor_SMD:R_0402_1005Metric
- R40, R49: value 120 -> 20k
- R48: value 2.2k -> 7.5k; footprint Resistor_SMD:R_0402_1005Metric -> Resistor_SMD:R_0603_1608Metric
- R50: value 120 -> 10k
Connections:
- net +3.3V: now also R24.1, R26.1, R33.1, R42.1, R44.1, R51.1, R53.1, C21.1, C22.1, Q5.2 (E), R79.1, R87.1, U14.8 (VCC), U16.8 (VCC); no longer R23.1, R28.1, R37.1, R45.1, R47.1, R55.1
- net at R40.1: now also Q8.3 (C), U6.2 (~{RE}), U6.3 (DE)
- net at U9.2 (~{RE}), U9.3 (DE): now also R50.1; no longer R54.1
- net at U8.2 (~{RE}), U8.3 (DE): now also Q9.3 (C), R49.1; no longer R53.1
- net at JP2.2 (B): now also R28.1; no longer R30.1
- net at Q7.1 (B): now also R30.1; no longer R26.1
- net at U5.2 (~{RE}), U5.3 (DE): now also R32.1; no longer Q9.3 (C), R34.1
- net RS485UI_B: now reaches R25.1
- net RS485UI_B: now also J2.4 (Pin_4), R28.2, U2.7 (B)
- net at U7.2 (~{RE}), U7.3 (DE): now also R41.1; no longer R44.1
- net GNDD: now reaches J5.1 (Pin_1)
- net GNDD: now also C11.2, C12.2, C13.2, C14.2, C15.2, C16.2, C17.2, C18.2, J2.1 (Pin_1), J2.MP (MountPin), J3.1 (Pin_1), J3.MP (MountPin), J4.1 (Pin_1), J4.MP (MountPin), J5.MP (MountPin), R22.2, R23.2, R25.2, R27.2, R31.2, R32.2, R34.2, R36.2, R40.2, R41.2, R43.2, R45.2, R49.2, R50.2, R52.2, R54.2, U2.5 (GND), U3.5 (GND), U4.5 (GND), U5.5 (GND), U6.5 (GND), U7.5 (GND), U8.5 (GND), U9.5 (GND), C21.2, C22.2, J8.1 (Pin_1), J8.MP (MountPin), R77.2, R78.2, R80.2, R88.2, U14.5 (GND), U16.5 (GND)
- net 24VOUT_Spr: now reaches J5.2 (Pin_2)
- net 24VOUT_Spr: now also JP15.2 (B)
- net RS485Spr_A: now reaches J5.3 (Pin_3)
- net RS485Spr_A: now also R51.2, U8.6 (A), JP13.1 (A)
- net RS485Spr_B: now reaches J5.4 (Pin_4)
- net RS485Spr_B: now also R52.1, R55.2, U8.7 (B)
- net RS485Spr_X: now reaches J5.5 (Pin_5)
- net RS485Spr_X: now also R53.2, U9.6 (A), JP14.1 (A)
- net RS485Spr_Y: now reaches J5.6 (Pin_6)
- net RS485Spr_Y: now also R54.1, R56.2, U9.7 (B)
- net at JP8.2 (B): now also R46.1
- net 24VOUT_Bst: now reaches J3.2 (Pin_2)
- net 24VOUT_Bst: now also JP7.2 (B)
- net RS485Bst_A: now reaches J3.3 (Pin_3)
- net RS485Bst_A: now also JP5.1 (A), R33.2, U4.6 (A)
- net RS485Bst_B: now reaches J3.4 (Pin_4)
- net RS485Bst_B: now also R34.1, R37.2, U4.7 (B)
- net RS485Bst_X: now reaches J3.5 (Pin_5)
- net RS485Bst_X: now also JP6.1 (A), R35.2, U5.6 (A)
- net RS485Bst_Y: now reaches J3.6 (Pin_6)
- net RS485Bst_Y: now also R36.1, R38.2, U5.7 (B)
- net at JP9.2 (B): now also R47.1
- net at R31.1: now also Q7.3 (C), U4.2 (~{RE}), U4.3 (DE); no longer Q8.1 (B)
- net 24VOUT_UI: now reaches J2.2 (Pin_2)
- net 24VOUT_UI: now also JP4.2 (B)
- net RS485UI_A: now reaches J2.3 (Pin_3)
- net RS485UI_A: now also JP2.1 (A), R24.2, U2.6 (A)
- net RS485UI_X: now reaches J2.5 (Pin_5)
- net RS485UI_X: now also JP3.1 (A), R26.2, U3.6 (A)
- net RS485UI_Y: now reaches J2.6 (Pin_6)
- net RS485UI_Y: now also R27.1, R29.2, U3.7 (B)
- net at JP6.2 (B): now also R38.1; no longer R50.1
- net at U3.2 (~{RE}), U3.3 (DE): now also R23.1; no longer Q7.3 (C), R27.1
- net 24VOUT_MD: now reaches J4.2 (Pin_2)
- net 24VOUT_MD: now also JP10.2 (B)
- net RS485MD_A: now reaches J4.3 (Pin_3)
- net RS485MD_A: now also JP8.1 (A), R42.2, U6.6 (A)
- net RS485MD_B: now reaches J4.4 (Pin_4)
- net RS485MD_B: now also R43.1, R46.2, U6.7 (B)
- net RS485MD_X: now reaches J4.5 (Pin_5)
- net RS485MD_X: now also JP9.1 (A), R44.2, U7.6 (A)
- net RS485MD_Y: now reaches J4.6 (Pin_6)
- net RS485MD_Y: now also R45.1, R47.2, U7.7 (B)
- net at JP5.2 (B): now also R37.1; no longer R49.1
- net at Q9.1 (B): now also R48.1; no longer R32.1
- net at JP3.2 (B): now also R29.1; no longer R39.1
- removed net GND: C11.2, C12.2, C13.2, C14.2, C15.2, C16.2, C17.2, C18.2, R22.2, R24.2, R27.2, R29.2, R33.2, R34.2, R36.2, R38.2, R43.2, R44.2, R46.2, R48.2, R53.2, R54.2, R56.2, U2.5 (GND), U3.5 (GND), U4.5 (GND), U5.5 (GND), U6.5 (GND), U7.5 (GND), U8.5 (GND), U9.5 (GND)
- removed net MainRX6_RS485aTX: U2.1 (RO), U3.1 (RO), U4.1 (RO), U5.1 (RO), U6.1 (RO), U7.1 (RO), U8.1 (RO), U9.1 (RO)
- removed net MainTX6_RS485aRX: R21.2, R26.2, R31.2, R32.2, R41.2, R42.2, R51.2, R52.2, U2.4 (DI), U3.4 (DI), U4.4 (DI), U5.4 (DI), U6.4 (DI), U7.4 (DI), U8.4 (DI), U9.4 (DI)
- removed net RS485a_A: JP2.1 (A), JP3.1 (A), JP5.1 (A), JP6.1 (A), JP8.1 (A), JP9.1 (A), R23.2, R28.2, R35.2, R37.2, R45.2, R47.2, R55.2, U2.6 (A), U3.6 (A), U4.6 (A), U5.6 (A), U6.6 (A), U7.6 (A), U8.6 (A), U9.6 (A)
- removed net RS485a_B: R24.1, R25.2, R29.1, R30.2, R36.1, R38.1, R39.2, R40.2, R46.1, R48.1, R49.2, R50.2, R56.1, U2.7 (B), U3.7 (B), U4.7 (B), U5.7 (B), U6.7 (B), U7.7 (B), U8.7 (B), U9.7 (B)
- new net: Q5.1 (B), R71.1
- new net: Q5.3 (C), R78.1, U16.2 (~{RE}), U16.3 (DE)
- new net: JP13.2 (B), R55.1
- new net: JP14.2 (B), R56.1
- new net: R77.1, U14.2 (~{RE}), U14.3 (DE)
- new net: JP12.2 (B), R90.1
- new net: JP11.2 (B), R89.1
- new net: Q8.1 (B), R39.1
- new net +BATT: JP1.1 (A), JP10.1 (A), JP15.1 (A), JP4.1 (A), JP7.1 (A)
- new net 24VOUT_Cam: J8.2 (Pin_2), JP1.2 (B)
- new net MainRX_RS485Bst_TX: U5.1 (RO)
- new net MainRX_RS485Cam_TX: U14.1 (RO)
- new net MainRX_RS485MD_TX: U7.1 (RO)
- new net MainRX_RS485Spr_TX: U9.1 (RO)
- new net MainRX_RS485UI_TX: U3.1 (RO)
- new net MainTX_RS485Bst_RX: R30.2, U4.4 (DI)
- new net MainTX_RS485Cam_RX: R71.2, U16.4 (DI)
- new net MainTX_RS485MD_RX: R39.2, U6.4 (DI)
- new net MainTX_RS485Spr_RX: R48.2, U8.4 (DI)
- new net MainTX_RS485UI_RX: R21.2, U2.4 (DI)
- new net RS485Cam_A: J8.3 (Pin_3), JP12.1 (A), R87.2, U16.6 (A)
- new net RS485Cam_B: J8.4 (Pin_4), R88.1, R90.2, U16.7 (B)
- new net RS485Cam_X: J8.5 (Pin_5), JP11.1 (A), R79.2, U14.6 (A)
- new net RS485cam_Y: J8.6 (Pin_6), R80.1, R89.2, U14.7 (B)
- no-connect marks 0 -> 10
Other:
- note added: "24V_conn"
- note added: "MAX3485_AB"
- note added: "MAX3485_XY"
- note added: "RS485_Bst"
- note added: "RS485_Camera"
- note added: "RS485_MD"
- note added: "RS485_Spare"
- note added: "RS485_UI"
- note removed: "MAX3485"
- note removed: "RS485a"

Commit message: とちゅう
Other:
- note added: "RS485_Bst/Host"
- note added: "RS485_Camera/Host"
- note added: "RS485_MD/Host"
- note added: "RS485_Spare/Host"
- note added: "RS485_UI/Host"
- note removed: "RS485_Bst"
- note removed: "RS485_Camera"
- note removed: "RS485_MD"
- note removed: "RS485_Spare"
- note removed: "RS485_UI"

Commit message: すてい
Parts:
- JP1, JP10, JP15, JP4, JP7: footprint (none) -> Jumper:SolderJumper-2_P1.3mm_Open_TrianglePad1.0x1.5mm
Connections:
- net 24VOUT_Bst: now also JP4.2 (B); no longer JP7.2 (B)
- net 24VOUT_MD: now also JP7.2 (B); no longer JP10.2 (B)
- net 24VOUT_UI: now also JP10.2 (B); no longer JP4.2 (B)
