File: circuits/Main/TweLite.kicad_sch (KiCad schematic)
At the start: 15 parts, among them J17 Conn_01x07_Female, Q10 BSS138, SW6 SW_SPST, SW7 SW_SPST, U15 TWE-L-WX

Commit message: すてい
Parts:
- removed R83, R84: 1k, Resistor_SMD:R_0402_1005Metric, symbol Device:R
- added R66, R67: 2k, Resistor_SMD:R_0402_1005Metric, symbol Device:R
Connections:
- net Twe_LED0: now also R66.2
- net Twe_LED1: now also R67.2
- net at D13.2 (A): now also R67.1
- net at D12.2 (A): now also R66.1
