File: circuits/Main/UI.kicad_sch (KiCad schematic)
At the start: 11 parts, among them SW2 SW_SPST, SW3 SW_SPDT, SW8 SW_SPDT

Commit message: すてい
Parts:
- R59, R60: value 1k -> 2k
Connections:
- net LED0: now also R60.2; no longer R59.2
- net LED1: now also R59.2; no longer R60.2
- net at R59.1: now also D11.2 (A); no longer D10.2 (A)
- net at R60.1: now also D10.2 (A); no longer D11.2 (A)
Changed lines of the file:
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@@
+    )
+  )
+  (symbol (lib_id "Device:R") (at 124.46 58.42 270) (mirror x) (unit 1)
+    (in_bom yes) (on_board yes) (dnp no)
+    (property "Reference" "R59" (at 124.46 63.5 90)
+      (effects (font (size 1.27 1.27)))
+    )
+    (property "Value" "2k" (at 124.46 60.96 90)
+      (effects (font (size 1.27 1.27)))
+    )
+    (property "Footprint" "Resistor_SMD:R_0402_1005Metric" (at 124.46 60.198 90)
+      (effects (font (size 1.27 1.27)) hide)
+    )
+    (property "Datasheet" "~" (at 124.46 58.42 0)
+      (effects (font (size 1.27 1.27)) hide)
+    )
+    (pin "1")
+    (pin "2")
+    (instances
+      (project "Main"
+        (path "/aa9d7141-7530-418f-853d-a56ee68433fb/2919e3e4-6b19-4436-850c-b08439974325"
+          (reference "R59") (unit 1)
+        )
+      )
     )
   )
@@
     )
   )
+  (symbol (lib_id "Device:R") (at 137.16 114.3 90) (mirror x) (unit 1)
+    (in_bom yes) (on_board yes) (dnp no)
+    (property "Reference" "R63" (at 139.7 116.84 90)
+      (effects (font (size 1.27 1.27)) (justify left))
+    )
+    (property "Value" "10k" (at 139.7 119.1514 90)
+      (effects (font (size 1.27 1.27)) (justify left))
+    )
+    (property "Footprint" "Resistor_SMD:R_0402_1005Metric" (at 137.16 112.522 90)
+      (effects (font (size 1.27 1.27)) hide)
+    )
+    (property "Datasheet" "~" (at 137.16 114.3 0)
+      (effects (font (size 1.27 1.27)) hide)
+    )
+    (pin "1")
+    (pin "2")
+    (instances
+      (project "Main"
+        (path "/aa9d7141-7530-418f-853d-a56ee68433fb/2919e3e4-6b19-4436-850c-b08439974325"
+          (reference "R63") (unit 1)
+        )
+      )
+    )
+  )
+  (symbol (lib_id "power:+3.3V") (at 114.3 132.08 0) (unit 1)
+    (in_bom yes) (on_board yes) (dnp no)
+    (property "Reference" "#PWR0135" (at 114.3 135.89 0)
+      (effects (font (size 1.27 1.27)) hide)
+    )
+    (property "Value" "+3.3V" (at 113.665 127.635 0)
+      (effects (font (size 1.27 1.27)))
+    )
+    (property "Footprint" "" (at 114.3 132.08 0)
+      (effects (font (size 1.27 1.27)) hide)
+    )
+    (property "Datasheet" "" (at 114.3 132.08 0)
+      (effects (font (size 1.27 1.27)) hide)
+    )
+    (pin "1")
+    (instances
+      (project "Main"
+        (path "/aa9d7141-7530-418f-853d-a56ee68433fb/2919e3e4-6b19-4436-850c-b08439974325"
+          (reference "#PWR0135") (unit 1)
+        )
+      )
+    )
+  )
   (symbol (lib_id "Device:R") (at 124.46 48.26 270) (mirror x) (unit 1)
     (in_bom yes) (on_board yes) (dnp no)
-    (property "Reference" "R59" (at 124.46 53.34 90)
-      (effects (font (size 1.27 1.27)))
-    )
-    (property "Value" "1k" (at 124.46 50.8 90)
+    (property "Reference" "R60" (at 124.46 53.34 90)
+      (effects (font (size 1.27 1.27)))
+    )
+    (property "Value" "2k" (at 124.46 50.8 90)
       (effects (font (size 1.27 1.27)))
     )
@@
       (effects (font (size 1.27 1.27)) hide)
     )
-    (pin "1")
-    (pin "2")
-    (instances
-      (project "Main"
-        (path "/aa9d7141-7530-418f-853d-a56ee68433fb/2919e3e4-6b19-4436-850c-b08439974325"
-          (reference "R59") (unit 1)
-        )
-      )
-    )
-  )
-  (symbol (lib_id "Device:R") (at 137.16 114.3 90) (mirror x) (unit 1)
-    (in_bom yes) (on_board yes) (dnp no)
-    (property "Reference" "R63" (at 139.7 116.84 90)
-      (effects (font (size 1.27 1.27)) (justify left))
-    )
-    (property "Value" "10k" (at 139.7 119.1514 90)
-      (effects (font (size 1.27 1.27)) (justify left))
-    )
-    (property "Footprint" "Resistor_SMD:R_0402_1005Metric" (at 137.16 112.522 90)
-      (effects (font (size 1.27 1.27)) hide)
-    )
-    (property "Datasheet" "~" (at 137.16 114.3 0)
-      (effects (font (size 1.27 1.27)) hide)
-    )
-    (pin "1")
-    (pin "2")
-    (instances
-      (project "Main"
-        (path "/aa9d7141-7530-418f-853d-a56ee68433fb/2919e3e4-6b19-4436-850c-b08439974325"
-          (reference "R63") (unit 1)
-        )
-      )
-    )
-  )
-  (symbol (lib_id "power:+3.3V") (at 114.3 132.08 0) (unit 1)
-    (in_bom yes) (on_board yes) (dnp no)
-    (property "Reference" "#PWR0135" (at 114.3 135.89 0)
-      (effects (font (size 1.27 1.27)) hide)
-    )
-    (property "Value" "+3.3V" (at 113.665 127.635 0)
-      (effects (font (size 1.27 1.27)))
-    )
-    (property "Footprint" "" (at 114.3 132.08 0)
-      (effects (font (size 1.27 1.27)) hide)
-    )
-    (property "Datasheet" "" (at 114.3 132.08 0)
-      (effects (font (size 1.27 1.27)) hide)
-    )
-    (pin "1")
-    (instances
-      (project "Main"
-        (path "/aa9d7141-7530-418f-853d-a56ee68433fb/2919e3e4-6b19-4436-850c-b08439974325"
-          (reference "#PWR0135") (unit 1)
-        )
-      )
-    )
-  )
-  (symbol (lib_id "Device:R") (at 124.46 58.42 270) (mirror x) (unit 1)
-    (in_bom yes) (on_board yes) (dnp no)
-    (property "Reference" "R60" (at 124.46 63.5 90)
-      (effects (font (size 1.27 1.27)))
-    )
-    (property "Value" "1k" (at 124.46 60.96 90)
-      (effects (font (size 1.27 1.27)))
-    )
-    (property "Footprint" "Resistor_SMD:R_0402_1005Metric" (at 124.46 60.198 90)
-      (effects (font (size 1.27 1.27)) hide)
-    )
-    (property "Datasheet" "~" (at 124.46 58.42 0)
-      (effects (font (size 1.27 1.27)) hide)
-    )
