File: circuits/UI/UserInterface.kicad_sch (KiCad schematic)
At the start: 44 parts, among them SW2 SW_SPDT, SW3 SW_SPDT, SW4 SW_SPDT, SW5 SW_SPST, SW6 SW_SPST, SW7 SW_SPST, U6 Display_Aktk_128x68OLED, U7 NJM4580C

Commit message: すてい
Parts:
- removed C22, C23: 10uF, Capacitor_SMD:C_0805_2012Metric, symbol Device:C
- removed C24, C25, C26, C27: 22uF, Capacitor_SMD:C_0805_2012Metric, symbol Device:C
- removed H4: MountingHole_Pad, TestPoint:TestPoint_Pad_1.5x1.5mm, symbol Mechanical:MountingHole_Pad
- removed R38: 5.1k, Resistor_SMD:R_0402_1005Metric, symbol Device:R
- removed R39, R40: 10k, Resistor_SMD:R_0402_1005Metric, symbol Device:R
- removed R41, R43: 5.1k, Resistor_SMD:R_0603_1608Metric, symbol Device:R
- removed R42, R44: 1k, Resistor_SMD:R_0603_1608Metric, symbol Device:R
- removed R45, R46: 47, Resistor_SMD:R_0603_1608Metric, symbol Device:R
- removed R48: 1k, Resistor_SMD:R_0402_1005Metric, symbol Device:R
- removed U7: NJM4580C, Package_SO:SOP-8_3.9x4.9mm_P1.27mm, symbol Amplifier_Operational:NJM4580
- added D10: 1N5819WS, Diode_SMD:D_SOD-323_HandSoldering, symbol Device:D_Schottky
- added Q7: BSS138, Package_TO_SOT_SMD:SOT-23, symbol Device:Q_NMOS_GSD
- R30, R31: value 1k -> 2k
- R37: value 5.1k -> 10k
Connections:
- net GNDD: now also R37.2, Q7.2 (S)
- net LED0: now also R31.2; no longer R30.2
- net LED1: now also R30.2; no longer R31.2
- net VCC: now also LS1.1, R47.1, D10.1 (K); no longer R37.2
- net at R31.1: now also D7.2 (A); no longer D8.2 (A)
- net at R30.1: now also D8.2 (A); no longer D7.2 (A)
- net GND: no longer names the net of LS1.2, R47.2
- net GND: now also D10.2 (A), Q7.3 (D)
- net GNDA renamed Speaker
- net Speaker: now also Q7.1 (G)
Other:
- note removed: "LEDのつよさをかえたい"
- note removed: "アンプ"
- note removed: "仮想GND"
- moved on the sheet: LS1, R47
