File: circuits/UI/Power.kicad_sch (KiCad schematic)
At the start: 47 parts, among them IC1 DCDC_MPM3620A, Q1 SSM6J808R, Q2 BSS138, Q3 SSM3J332R, Q4 BSS138, Q5 SSM6J808R, SW1 SW_SPDT_White, U1 AZ1117CH-3.3

Commit message: すてい
Parts:
- R19, R20: value 1k -> 2k
Changed lines of the file:
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@@
       (effects (font (size 1.27 1.27)))
     )
-    (property "Value" "1k" (at 251.46 137.16 90)
+    (property "Value" "2k" (at 251.46 137.16 90)
       (effects (font (size 1.27 1.27)))
     )
@@
     )
   )
+  (symbol (lib_id "Device:R") (at 251.46 147.32 270) (mirror x) (unit 1)
+    (in_bom yes) (on_board yes) (dnp no)
+    (property "Reference" "R20" (at 251.46 152.4 90)
+      (effects (font (size 1.27 1.27)))
+    )
+    (property "Value" "2k" (at 251.46 149.86 90)
+      (effects (font (size 1.27 1.27)))
+    )
+    (property "Footprint" "Resistor_SMD:R_0402_1005Metric" (at 251.46 149.098 90)
+      (effects (font (size 1.27 1.27)) hide)
+    )
+    (property "Datasheet" "~" (at 251.46 147.32 0)
+      (effects (font (size 1.27 1.27)) hide)
+    )
+    (pin "1")
+    (pin "2")
+    (instances
+      (project "UI"
+        (path "/cc146f76-4a67-4abf-9b83-f5188f4bdf5e/7479307e-135d-4549-8171-4a735831bfb8"
+          (reference "R20") (unit 1)
+        )
+      )
+    )
+  )
   (symbol (lib_id "Device:R") (at 88.9 147.32 180) (unit 1)
     (in_bom yes) (on_board yes) (dnp no)
@@
         )
       )
-    )
-  )
-  (symbol (lib_id "Device:R") (at 251.46 147.32 270) (mirror x) (unit 1)
-    (in_bom yes) (on_board yes) (dnp no)
-    (property "Reference" "R20" (at 251.46 152.4 90)
-      (effects (font (size 1.27 1.27)))
-    )
-    (property "Value" "1k" (at 251.46 149.86 90)
-      (effects (font (size 1.27 1.27)))
-    )
-    (property "Footprint" "Resistor_SMD:R_0402_1005Metric" (at 251.46 149.098 90)
-      (effects (font (size 1.27 1.27)) hide)
-    )
-    (property "Datasheet" "~" (at 251.46 147.32 0)
-      (effects (font (size 1.27 1.27)) hide)
-    )
-    (pin "1")
-    (pin "2")
-    (instances
-      (project "UI"
-        (path "/cc146f76-4a67-4abf-9b83-f5188f4bdf5e/7479307e-135d-4549-8171-4a735831bfb8"
-          (reference "R20") (unit 1)
-        )
-      )

Commit message: 修正
Other:
- note added: "電源スイッチ 耐圧大丈夫？"
Changed lines of the file:
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@@
     (effects (font (size 1.27 1.27)) (justify left bottom))
+  )
+  (text "電源スイッチ　耐圧大丈夫？" (at 121.92 20.32 0)
+    (effects (font (size 5.56 5.56)) (justify left bottom))
   )
   (text "5V生成" (at 27.94 109.22 0)
