File: circuits/UI/UI.kicad_sch (KiCad schematic)
At the start: 11 parts, among them J4 Conn_01x04_Female, SW8 SW_SPST, U5 STM32C011F6P6, Y1 48MHz

Commit message: すてい
Parts:
- removed H2: UART1_TX, TestPoint:TestPoint_Pad_1.5x1.5mm, symbol Mechanical:MountingHole_Pad
- removed H3: UART1_RX, TestPoint:TestPoint_Pad_1.5x1.5mm, symbol Mechanical:MountingHole_Pad
- added D9: 1N5819WS, Diode_SMD:D_SOD-323_HandSoldering, symbol Device:D_Schottky
- added J1: Conn_01x14_Pin, MyLibrary:BoxHeader_2x07_P1.27mm_Horizontal, symbol Connector:Conn_01x14_Pin
- added R52: 1k, Resistor_SMD:R_0402_1005Metric, symbol Device:R
Connections:
- net +3.3V: now also D9.2 (A)
- net GNDD: now also J1.11 (Pin_11), J1.5 (Pin_5), J1.7 (Pin_7), R52.2
- net NRST: now also J1.12 (Pin_12)
- net MainRX1_RS485TX: now reaches U5.8 (PA1)
- net MainTX1_RS485RX: now reaches U5.7 (PA0)
- net DIP_SW0: no longer names the net of U5.12 (PA5)
- net DIP_SW1: no longer names the net of U5.13 (PA6)
- net DIP_SW2: no longer names the net of U5.14 (PA7)
- net DIP_SW3: no longer names the net of U5.15 (PA8)
- net DIP_SW4: no longer names the net of U5.16 (PA11[PA9])
- net MainRX2_RS485TX: no longer names the net of U5.10 (PA3)
- net MainTX2_RS485RX: no longer names the net of U5.9 (PA2)
- net MonitorLED0: no longer names the net of U5.11 (PA4)
- net TCK renamed SWCLK
- net SWCLK: now also J1.6 (Pin_6)
- net TMS renamed SWDIO
- net SWDIO: now also J1.4 (Pin_4)
- new net: D9.1 (K), J1.3 (Pin_3), R52.1
- no-connect marks 1 -> 7
Other:
- sheet Power ports: added V_Meas.; removed none
- sheet RS485 ports: added MainRX_RS485TX, MainTX_RS485RX; removed none
- sheet UserInterface ports: added I2C_SCL, I2C_SDA, LED0, LED1, Slide_SW0, Slide_SW1, Speaker, Tact_SW0, Tact_SW1, Tact_SW2, Toggle_SW0; removed none
- note added: "V3"
- note added: "オシレーターの周波数とフットプリント"
- moved on the sheet: C18, C19, C20, C21, H1, J4, SW8, U5, Y1

Commit message: 修正
Other:
- note added: "オシレーターの周波数とフットプリント 電解コンの耐圧注意"
- note removed: "オシレーターの周波数とフットプリント"
Changed lines of the file:
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@@
     (effects (font (size 1.27 1.27)) (justify left bottom))
   )
-  (text "オシレーターの周波数とフットプリント" (at 104.14 38.1 0)
+  (text "オシレーターの周波数とフットプリント\n電解コンの耐圧注意" (at 104.14 38.1 0)
     (effects (font (size 5.56 5.56)) (justify left bottom))
   )
