File: circuits/Boost/Boost.kicad_sch (KiCad schematic)
At the start: 12 parts, among them J6 Conn_01x04_Female, J7 Conn_01x14_Pin, SW2 SW_SPST, U2 STM32C011F6P6, Y1 48MHz

Commit message: 修正
Other:
- note added: "オシレーターの周波数とフットプリント キック回路のハイサイドは電圧制限でNchでブートストラップできない問題 昇圧の目標値は45V位にしよう 電解コンの耐圧注意"
- note removed: "オシレーターの周波数とフットプリント キック回路のハイサイドは電圧制限でNchでブートストラップできない問題 昇圧の目標値は45V位にしよう"
Changed lines of the file:
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@@
     (effects (font (size 1.27 1.27)) (justify left bottom))
   )
-  (text "オシレーターの周波数とフットプリント\nキック回路のハイサイドは電圧制限でNchでブートストラップできない問題\n昇圧の目標値は45V位にしよう"
+  (text "オシレーターの周波数とフットプリント\nキック回路のハイサイドは電圧制限でNchでブートストラップできない問題\n昇圧の目標値は45V位にしよう\n電解コンの耐圧注意"
     (at 109.22 35.56 0)
     (effects (font (size 5.56 5.56)) (justify left bottom))
