File: circuits/Boost/Power.kicad_sch (KiCad schematic)
At the start: 48 parts, among them IC1 DCDC_MPM3620A, J1 Conn_01x02_Male, Q1 DI035P04PT, Q2 BSS138, Q3 SSM3J332R, Q4 BSS138, Q5 DI035P04PT, SW1 SW_SPDT_White, U1 AZ1117CH-3.3

Commit message: 修正
Other:
- note added: "電源スイッチ 耐圧大丈夫？"
Changed lines of the file:
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@@
     (effects (font (size 1.27 1.27)) (justify left bottom))
+  )
+  (text "電源スイッチ　耐圧大丈夫？" (at 104.14 20.32 0)
+    (effects (font (size 5.56 5.56)) (justify left bottom))
   )
   (text "Conn to Power" (at 20.32 33.02 0)
