File: circuits/Power/Power.kicad_sch (KiCad schematic)
At the start: 20 parts, among them J2 Conn_01x02_Male, J3 Conn_01x02_Socket, Q1 SQS141ELNW, Q4 BSS138, Q5 SQS141ELNW, SW1 SW_SPST

Commit message: 修正
Other:
- note added: "電解コンの耐圧注意"
Changed lines of the file:
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@@
     (effects (font (size 1.27 1.27)) (justify left bottom))
+  )
+  (text "電解コンの耐圧注意" (at 137.16 40.64 0)
+    (effects (font (size 5.56 5.56)) (justify left bottom))
   )
   (text "PowerModule" (at 40.64 60.96 0)
